Commit message: lasede

File: src/robot_square/robot_square/urdf/robot.urdf (robot description, URDF)
Before this commit: robot planar_arm, 5 links, 4 joints
Links:
- link base_link: mass None -> 1.0
- link end_effector: mass None -> 0.2
- link link1: mass None -> 1.0
- link link2: mass None -> 1.0
- link link3: mass None -> 1.0
Joints:
- joint joint1: axis 0 1 0 -> 0 0 1
- joint joint2: axis 0 1 0 -> 0 0 1
- joint joint3: axis 0 1 0 -> 0 0 1
